Commit message: Add Piper inspection ready postures

File: src/agx_arm_moveit/config/agx_arm.srdf.xacro (robot description, xacro)
@@ -348,4 +348,44 @@
       <joint name="joint6" value="0" />
     </group_state>
+    <group_state name="inspection_ready" group="arm">
+      <joint name="joint1" value="-0.0235619449" />
+      <joint name="joint2" value="1.9081684712" />
+      <joint name="joint3" value="-0.9113585755" />
+      <joint name="joint4" value="0.0" />
+      <joint name="joint5" value="-0.3634124569" />
+      <joint name="joint6" value="0.0" />
+    </group_state>
+    <group_state name="inspection_ready_yaw_left" group="arm">
+      <joint name="joint1" value="0.0964380551" />
+      <joint name="joint2" value="1.9081684712" />
+      <joint name="joint3" value="-0.9113585755" />
+      <joint name="joint4" value="0.0" />
+      <joint name="joint5" value="-0.3634124569" />
+      <joint name="joint6" value="0.0" />
+    </group_state>
+    <group_state name="inspection_ready_yaw_right" group="arm">
+      <joint name="joint1" value="-0.1435619449" />
+      <joint name="joint2" value="1.9081684712" />
+      <joint name="joint3" value="-0.9113585755" />
+      <joint name="joint4" value="0.0" />
+      <joint name="joint5" value="-0.3634124569" />
+      <joint name="joint6" value="0.0" />
+    </group_state>
+    <group_state name="inspection_ready_roll_left" group="arm">
+      <joint name="joint1" value="-0.0235619449" />
+      <joint name="joint2" value="1.9081684712" />
+      <joint name="joint3" value="-0.9113585755" />
+      <joint name="joint4" value="0.0" />
+      <joint name="joint5" value="-0.3634124569" />
+      <joint name="joint6" value="0.12" />
+    </group_state>
+    <group_state name="inspection_ready_roll_right" group="arm">
+      <joint name="joint1" value="-0.0235619449" />
+      <joint name="joint2" value="1.9081684712" />
+      <joint name="joint3" value="-0.9113585755" />
+      <joint name="joint4" value="0.0" />
+      <joint name="joint5" value="-0.3634124569" />
+      <joint name="joint6" value="-0.12" />
+    </group_state>
   </xacro:unless>
   <xacro:if value="$(eval arm_type == 'nero')">

Commit message: [Dev] LRC Freeze
Signed-off-by: Bichy <bichyzhang@gmail.com>

File: src/agx_arm_moveit/config/agx_arm.srdf.xacro (robot description, xacro)
@@ -388,4 +388,28 @@
       <joint name="joint6" value="-0.12" />
     </group_state>
+    <group_state name="inspection_ready_far" group="arm">
+      <joint name="joint1" value="-0.0235619449" />
+      <joint name="joint2" value="1.6081684712" />
+      <joint name="joint3" value="-0.7613585755" />
+      <joint name="joint4" value="0.0" />
+      <joint name="joint5" value="-0.2134124569" />
+      <joint name="joint6" value="0.0" />
+    </group_state>
+    <group_state name="inspection_ready_far_yaw_left" group="arm">
+      <joint name="joint1" value="0.0964380551" />
+      <joint name="joint2" value="1.6081684712" />
+      <joint name="joint3" value="-0.7613585755" />
+      <joint name="joint4" value="0.0" />
+      <joint name="joint5" value="-0.2134124569" />
+      <joint name="joint6" value="0.0" />
+    </group_state>
+    <group_state name="inspection_ready_far_yaw_right" group="arm">
+      <joint name="joint1" value="-0.1435619449" />
+      <joint name="joint2" value="1.6081684712" />
+      <joint name="joint3" value="-0.7613585755" />
+      <joint name="joint4" value="0.0" />
+      <joint name="joint5" value="-0.2134124569" />
+      <joint name="joint6" value="0.0" />
+    </group_state>
   </xacro:unless>
   <xacro:if value="$(eval arm_type == 'nero')">
